Commit message: Add files via upload

File: AgriBot/config/gazebo_roarm_assembly.urdf (robot description, URDF)
Before this commit: robot roarm_assembly, 7 links, 6 joints
Links:
- added link world
Joints:
- added joint base_fixed: type fixed, parent world, child base_link, origin xyz=0.0 0.0 0.0 rpy=0.0 0.0 0.0
